File: ESP32_Devkit_TypeC.kicad_sch (KiCad schematic)
At the start: 63 parts, among them Q1 MMBT3904, Q2 MMBT3904, U2 CH340C, Y2 40MHz

Commit message: Layout revision F
Parts:
- AE1: value (none) -> Antenna_Shield; footprint (none) -> Antenna_IFA:Antenna_IFA_2.4GHz_meandered
- C1: value (none) -> 22nF; footprint (none) -> Capacitor_SMD:C_0402_1005Metric
- C10, C11, C27, C28, C9: value (none) -> DNP; footprint (none) -> Capacitor_SMD:C_0402_1005Metric
- C12, C13: value (none) -> 30pF; footprint (none) -> Capacitor_SMD:C_0402_1005Metric
- C14: value (none) -> 10uF; footprint (none) -> Capacitor_SMD:C_0402_1005Metric
- C15, C16, C17, C26: value (none) -> 1uF; footprint (none) -> Capacitor_SMD:C_0402_1005Metric
- C18: value (none) -> 3.3nF; footprint (none) -> Capacitor_SMD:C_0402_1005Metric
- C19, C5: value (none) -> 10nF; footprint (none) -> Capacitor_SMD:C_0402_1005Metric
- C20, C21, C24, C25, C7: value (none) -> 100nF; footprint (none) -> Capacitor_SMD:C_0402_1005Metric
- C22: value (none) -> 100pF; footprint (none) -> Capacitor_SMD:C_0402_1005Metric
- C3: value (none) -> 10uF 25V; footprint (none) -> Capacitor_SMD:C_0805_2012Metric; LCSC C45783 -> C15850
- C6, C8: value (none) -> 22uF; footprint (none) -> Capacitor_SMD:C_0603_1608Metric
- D1: value (none) -> B5819W; footprint (none) -> Diode_SMD:D_SOD-123
- D2, D3: value (none) -> LED; footprint (none) -> LED_SMD:LED_0603_1608Metric_Castellated
- H1, H2: value (none) -> MountingHole; footprint (none) -> ToolingHole:ToolingHole_JLCSMT
- I2: value (none) -> Icon; footprint (none) -> Signs:OSHW_icon_3.3x3
- J1: value (none) -> USB_C_Receptacle_USB2.0; footprint (none) -> Connector_USB:USB_C_Receptacle_Palconn_UTC16-G
- J2, J3: value (none) -> Conn_01x19; footprint (none) -> Connector_PinHeader_2.54mm:PinHeader_1x19_P2.54mm_Vertical
- JP1: value (none) -> SolderJumper_2_Open; footprint (none) -> Jumper:SolderJumper-2_P1.3mm_Open_Pad1.0x1.5mm
- L1: value 10uH -> 4.7uH; LCSC C701155 -> C90319
- L2: value (none) -> 4.7nH; footprint (none) -> Inductor_SMD:L_0603_1608Metric
- L3: value (none) -> 0R; footprint (none) -> Inductor_SMD:L_0402_1005Metric
- R1, R10, R5: value (none) -> 100k; footprint (none) -> Resistor_SMD:R_0402_1005Metric
- R11, R12, R4: value (none) -> 330R; footprint (none) -> Resistor_SMD:R_0402_1005Metric
- R13: value (none) -> 20k; footprint (none) -> Resistor_SMD:R_0402_1005Metric
- R14, R2, R3, R7, R8, R9: value (none) -> 5.1k; footprint (none) -> Resistor_SMD:R_0402_1005Metric
- R6: value (none) -> 22k; footprint (none) -> Resistor_SMD:R_0402_1005Metric
- SW1: value (none) -> EN; footprint (none) -> Button_Switch_SMD:SW_Push_SPST_NO_Alps_SKRK
- SW2: value (none) -> BOOT; footprint (none) -> Button_Switch_SMD:SW_Push_SPST_NO_Alps_SKRK
- U1: value (none) -> SD8942; footprint (none) -> Package_TO_SOT_SMD:SOT-23-6
- U3: value (none) -> W25Q128JVS; footprint (none) -> Package_SO:SOIC-8_5.23x5.23mm_P1.27mm
- U4: value (none) -> ESP32-D0WD; footprint (none) -> Package_DFN_QFN:QFN-48-1EP_5x5mm_P0.35mm_EP3.7x3.7mm_ThermalVias; LCSC (none) -> C967020

Commit message: Add pin header partnumber
Parts:
- AE1: footprint Antenna_IFA:Antenna_IFA_2.4GHz_meandered -> Antenna_IFA:Antenna_IFA_2.4GHz_meandered_mirrored
- J2, J3: LCSC (none) -> C2894942
Changed lines of the file:
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@@
+      (effects (font (size 1.27 1.27)) hide)
+    )
+    (property "LCSC" "C2894942" (id 4) (at -58.42 66.04 0)
       (effects (font (size 1.27 1.27)) hide)
     )
@@
       (effects (font (size 1.27 1.27)) hide)
     )
+    (property "LCSC" "C2894942" (id 4) (at 322.58 113.03 0)
+      (effects (font (size 1.27 1.27)) hide)
+    )
     (pin "1")
     (pin "10")
@@
       (effects (font (size 1.27 1.27)) (justify left))
     )
-    (property "Footprint" "Antenna_IFA:Antenna_IFA_2.4GHz_meandered" (id 2) (at 264.16 67.31 0)
+    (property "Footprint" "Antenna_IFA:Antenna_IFA_2.4GHz_meandered_mirrored" (id 2) (at 264.16 67.31 0)
       (effects (font (size 1.27 1.27)) hide)
     )
@@
     )
     (path "/00000000-0000-0000-0000-00005f1a8ada"
-      (reference "AE1") (unit 1) (value "Antenna_Shield") (footprint "Antenna_IFA:Antenna_IFA_2.4GHz_meandered")
+      (reference "AE1") (unit 1) (value "Antenna_Shield") (footprint "Antenna_IFA:Antenna_IFA_2.4GHz_meandered_mirrored")
     )
     (path "/00000000-0000-0000-0000-000061df4449"

Commit message: Remove stray pin1 dot
Parts:
- C27: footprint Capacitor_SMD:C_0402_1005Metric -> L3
- L3: LCSC (none) -> C17168
Changed lines of the file:
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@@
+      (effects (font (size 1.27 1.27)) hide)
+    )
+    (property "LCSC" "C17168" (id 4) (at 259.08 82.55 90)
       (effects (font (size 1.27 1.27)) hide)
     )
@@
       (effects (font (size 1.27 1.27)) (justify right))
     )
-    (property "Footprint" "Capacitor_SMD:C_0402_1005Metric" (id 2) (at 254 86.36 0)
+    (property "Footprint" "L3" (id 2) (at 254 86.36 0)
       (effects (font (size 1.27 1.27)) hide)
     )
@@
     )
     (path "/00000000-0000-0000-0000-000062901d6f"
-      (reference "C27") (unit 1) (value "DNP") (footprint "Capacitor_SMD:C_0402_1005Metric")
+      (reference "C27") (unit 1) (value "DNP") (footprint "L3")
     )
     (path "/00000000-0000-0000-0000-0000629c777f"
